Commit message: Launch arg/path fixed.

File: f1tenth_vehicle_description/urdf/vehicle.xacro (robot description, xacro)
@@ -1,6 +1,8 @@
 <?xml version="1.0"?>
 <robot xmlns:xacro="http://ros.org/wiki/xacro">
+  <xacro:arg name="vehicle_model" default="f1tenth_vehicle"/>
+  <xacro:property name="vehicle_model_property" value="$(arg vehicle_model)"/>
   <!-- load parameter -->
-  <xacro:property name="vehicle_info" value="${xacro.load_yaml('$(find sample_vehicle_description)/config/vehicle_info.param.yaml')}"/>
+  <xacro:property name="vehicle_info" value="${xacro.load_yaml('$(find ${vehicle_model_property}_description)/config/vehicle_info.param.yaml')}"/>
   <!-- vehicle body -->
   <link name="base_link">
@@ -8,5 +10,5 @@
       <origin xyz="${vehicle_info['/**']['ros__parameters']['wheel_base']/2.0} 0 0" rpy="${pi/2.0} 0 ${pi}"/>
       <geometry>
-        <mesh filename="package://sample_vehicle_description/mesh/lexus.dae" scale="1 1 1"/>
+        <mesh filename="package://${vehicle_model_property}_description/mesh/lexus.dae" scale="1 1 1"/>
       </geometry>
     </visual>

Commit message: Launch arg/path fixed.

File: f1tenth_vehicle_description/urdf/vehicle.xacro (robot description, xacro)
@@ -1,8 +1,6 @@
 <?xml version="1.0"?>
 <robot xmlns:xacro="http://ros.org/wiki/xacro">
-  <xacro:arg name="vehicle_model" default="f1tenth_vehicle"/>
-  <xacro:property name="vehicle_model_property" value="$(arg vehicle_model)"/>
   <!-- load parameter -->
-  <xacro:property name="vehicle_info" value="${xacro.load_yaml('$(find ${vehicle_model_property}_description)/config/vehicle_info.param.yaml')}"/>
+  <xacro:property name="vehicle_info" value="${xacro.load_yaml('$(find f1tenth_vehicle_description)/config/vehicle_info.param.yaml')}"/>
   <!-- vehicle body -->
   <link name="base_link">
@@ -10,5 +8,5 @@
       <origin xyz="${vehicle_info['/**']['ros__parameters']['wheel_base']/2.0} 0 0" rpy="${pi/2.0} 0 ${pi}"/>
       <geometry>
-        <mesh filename="package://${vehicle_model_property}_description/mesh/lexus.dae" scale="1 1 1"/>
+        <mesh filename="package://f1tenth_vehicle_description/mesh/lexus.dae" scale="1 1 1"/>
       </geometry>
     </visual>

Commit message: Added rear axle link.

File: f1tenth_vehicle_description/urdf/vehicle.xacro (robot description, xacro)
@@ -12,3 +12,9 @@
     </visual>
   </link>
+  <joint name="rear_axle_joint" type="fixed">
+    <origin xyz="0 0 ${vehicle_info['/**']['ros__parameters']['wheel_radius']}" rpy="0 0 0"/>
+    <parent link="base_link"/>
+    <child link="rear_axle"/>
+  </joint>
+  <link name="rear_axle"/>
 </robot>
